Commit message: medidas correctas

File: armurdf2/urdf/armurdf2.urdf (robot description, URDF)
Before this commit: robot ROBOTARMURDF, 5 links, 4 joints
Links:
- link base_link: geometry collision mesh filename=package://armurdf2/meshes/base_link.STL; visual mesh filename=package://armurdf2/meshes/base_link.STL
- link link1: geometry collision mesh filename=package://armurdf2/meshes/link1.STL; visual mesh filename=package://armurdf2/meshes/link1.STL
- link link2: geometry collision mesh filename=package://armurdf2/meshes/link2.STL; visual mesh filename=package://armurdf2/meshes/link2.STL
- link link3: geometry collision mesh filename=package://armurdf2/meshes/link3.STL; visual mesh filename=package://armurdf2/meshes/link3.STL
- link link4: geometry collision mesh filename=package://armurdf2/meshes/link4.STL; visual mesh filename=package://armurdf2/meshes/link4.STL
Joints:
- joint joint2: limit lower=-1.57 upper=1.57 effort=120 velocity=3 -> lower=-1.57 upper=1.309 effort=120 velocity=3
- joint joint3: axis 0 0 -1 -> 0 0 1; limit lower=1.57 upper=-1.57 effort=40 velocity=2.2 -> lower=-1.57 upper=1.0472 effort=40 velocity=2.2
- joint joint4: limit lower=0 upper=-3.14 effort=27 velocity=2.3 -> lower=-3.14 upper=3.14 effort=27 velocity=2.3
